Commit message: Added simulation notes and launch files.

File: controlko_description/urdf/common.xacro (robot description, xacro)
@@ -19,10 +19,22 @@
   <material name="StoglRobotics/Violet">
     <color rgba="${102/255} ${46/255} ${145/255} 1.0"/>
+    <ambient>1 0 0 1</ambient>
+    <diffuse>1 0 0 1</diffuse>
+    <specular>0.1 0.1 0.1 1</specular>
+    <emissive>0 0 0 0</emissive>
   </material>
   <material name="StoglRobotics/DarkGrey">
     <color rgba="${51/255} ${51/255} ${51/255} 1.0"/>
+    <ambient>1 0 0 1</ambient>
+    <diffuse>1 0 0 1</diffuse>
+    <specular>0.1 0.1 0.1 1</specular>
+    <emissive>0 0 0 0</emissive>
   </material>
   <material name="StoglRobotics/LightGrey">
     <color rgba="${194/255} ${194/255} ${194/255} 1.0"/>
+    <ambient>1 0 0 1</ambient>
+    <diffuse>1 0 0 1</diffuse>
+    <specular>0.1 0.1 0.1 1</specular>
+    <emissive>0 0 0 0</emissive>
   </material>
 </robot>

File: controlko_description/urdf/rrbot.urdf.xacro (robot description, xacro)
@@ -2,7 +2,10 @@
 <robot xmlns:xacro="http://wiki.ros.org/xacro" name="rrbot">
   <!-- Use this if parameters are set from the launch file, otherwise delete -->
+  <xacro:arg name="prefix" default="" />
   <xacro:arg name="use_mock_hardware" default="false" />
   <xacro:arg name="mock_sensor_commands" default="false" />
-  <xacro:arg name="prefix" default="" />
+  <xacro:arg name="sim_gazebo_classic" default="false" />
+  <xacro:arg name="sim_gazebo" default="false" />
+  <xacro:arg name="simulation_controllers" default="" />
   <xacro:include filename="$(find controlko_description)/urdf/rrbot/rrbot_macro.xacro"/>
   <xacro:include filename="$(find controlko_description)/urdf/rrbot/rrbot_macro.ros2_control.xacro"/>
@@ -18,4 +21,27 @@
     prefix="$(arg prefix)"
     use_mock_hardware="$(arg use_mock_hardware)"
-    mock_sensor_commands="$(arg mock_sensor_commands)" />
+    mock_sensor_commands="$(arg mock_sensor_commands)"
+    sim_gazebo_classic="$(arg sim_gazebo_classic)"
+    sim_gazebo="$(arg sim_gazebo)"/>
+  <xacro:if value="$(arg sim_gazebo_classic)">
+    <!-- Gazebo plugins -->
+    <gazebo reference="world">
+    </gazebo>
+    <gazebo>
+      <plugin filename="libgazebo_ros2_control.so" name="gazebo_ros2_control">
+        <parameters>$(arg simulation_controllers)</parameters>
+      </plugin>
+    </gazebo>
+  </xacro:if>
+  <xacro:if value="$(arg sim_gazebo)">
+    <!-- Gazebo plugins -->
+    <gazebo reference="world">
+    </gazebo>
+    <gazebo>
+      <plugin filename="libign_ros2_control-system.so" name="ign_ros2_control::IgnitionROS2ControlPlugin">
+        <parameters>$(arg simulation_controllers)</parameters>
+        <controller_manager_node_name>$(arg prefix)controller_manager</controller_manager_node_name>
+      </plugin>
+    </gazebo>
+  </xacro:if>
 </robot>

File: controlko_description/urdf/rrbot/rrbot_macro.ros2_control.xacro (robot description, xacro)
@@ -1,29 +1,48 @@
 <?xml version="1.0" encoding="UTF-8"?>
 <robot xmlns:xacro="http://wiki.ros.org/xacro">
-  <xacro:macro name="rrbot_ros2_control" params="name prefix use_mock_hardware:=^|false mock_sensor_commands:=^|false">
+  <xacro:macro name="rrbot_ros2_control" params="
+               name
+               prefix
+               use_mock_hardware:=^|false
+               mock_sensor_commands:=^|false
+               sim_gazebo_classic:=^|false
+               sim_gazebo:=^|false"
+               >
     <ros2_control name="${name}" type="system">
       <hardware>
-        <plugin>mock_components/GenericSystem</plugin>
-        <param name="mock_sensor_commands">${mock_sensor_commands}</param>
+        <xacro:if value="${use_mock_hardware}">
+          <plugin>mock_components/GenericSystem</plugin>
+          <param name="mock_sensor_commands">${mock_sensor_commands}</param>
+        </xacro:if>
+        <xacro:if value="${sim_gazebo_classic}">
+          <plugin>gazebo_ros2_control/GazeboSystem</plugin>
+        </xacro:if>
+        <xacro:if value="${sim_gazebo}">
+          <plugin>ign_ros2_control/IgnitionSystem</plugin>
+        </xacro:if>
       </hardware>
       <joint name="${prefix}joint1">
-        <command_interface name="position">
-          <param name="min">-1</param>
-          <param name="max">1</param>
-        </command_interface>
-        <state_interface name="position"/>
-        <state_interface name="velocity"/>
-        <state_interface name="acceleration"/>
-        <param name="initial_position">0.0</param>
+        <command_interface name="position"/>
+        <state_interface name="position">
+          <param name="initial_value">0.0</param>
+        </state_interface>
+        <state_interface name="velocity">
+          <param name="initial_value">0.0</param>
+        </state_interface>
+        <state_interface name="effort">
+          <param name="initial_value">0.0</param>
+        </state_interface>
       </joint>
       <joint name="${prefix}joint2">
-        <command_interface name="position">
-          <param name="min">-1</param>
-          <param name="max">1</param>
-        </command_interface>
-        <state_interface name="position"/>
-        <state_interface name="velocity"/>
-        <state_interface name="acceleration"/>
-        <param name="initial_position">0.0</param>
+        <command_interface name="position"/>
+        <state_interface name="position">
+          <param name="initial_value">0.0</param>
+        </state_interface>
+        <state_interface name="velocity">
+          <param name="initial_value">0.0</param>
+        </state_interface>
+        <state_interface name="effort">
+          <param name="initial_value">0.0</param>
+        </state_interface>
       </joint>
       <sensor name="tcp_fts_sensor">

File: controlko_description/urdf/rrbot/rrbot_macro.xacro (robot description, xacro)
@@ -13,5 +13,4 @@
         <geometry>
           <box size="0.3 0.3 0.3"/>
-<!--           <mesh filename="package://controlko_description/meshes/rrbot/visual/base_link.dae" /> -->
         </geometry>
         <material name="StoglRobotics/Violet"/>
@@ -21,8 +20,10 @@
         <geometry>
           <box size="0.3 0.3 0.3"/>
-<!--           <mesh filename="package://controlko_description/meshes/rrbot/collision/base_link.stl" /> -->
         </geometry>
       </collision>
     </link>
+    <gazebo reference="${prefix}base_link">
+      <material>Gazebo/Orange</material>
+    </gazebo>
     <!-- link 1 -->
     <link name="${prefix}link1">
@@ -44,4 +45,7 @@
       </collision>
     </link>
+    <gazebo reference="${prefix}link1">
+        <material>Gazebo/Black</material>
+    </gazebo>
     <!-- link 2 -->
     <link name="${prefix}link2">
@@ -63,4 +67,7 @@
       </collision>
     </link>
+    <gazebo reference="${prefix}link2">
+      <material>Gazebo/Gray</material>
+    </gazebo>
     <!-- All-zero tool frame. This frame should correspond to the TOOL frame of the robot's controller.) -->
     <link name="${prefix}tool0" />
@@ -88,5 +95,5 @@
       <child link="${prefix}link1" />
       <axis xyz="0 0 1" />
-      <limit effort="0" lower="${radians(-380)}" upper="${radians(380)}" velocity="${radians(180)}" />
+      <limit effort="1000" lower="${radians(-380)}" upper="${radians(380)}" velocity="${radians(180)}" />
     </joint>
     <!-- joint 2 -->
@@ -96,5 +103,5 @@
       <child link="${prefix}link2" />
       <axis xyz="0 1 0" />
-      <limit effort="0" lower="${radians(-60)}" upper="${radians(240)}" velocity="${radians(180)}" />
+      <limit effort="1000" lower="${radians(-60)}" upper="${radians(240)}" velocity="${radians(180)}" />
     </joint>
     <!-- tool frame - fixed frame -->
